Commit message: Implemented voxel description

File: src/floatbot_description/urdf/floatbot.urdf.xacro (robot description, xacro)
@@ -4,6 +4,12 @@
     <xacro:arg name="prefix" default=""/>
     <xacro:include filename="$(find floatbot_description)/urdf/floatbot_base.urdf.xacro"/>
+    <xacro:include filename="$(find floatbot_description)/urdf/voxel.urdf.xacro"/>
     <xacro:floatbot_base
         prefix="$(arg prefix)"
     />
+    <xacro:voxel
+        prefix="$(arg prefix)"
+        parent="$(arg prefix)base_link">
+        <origin xyz="0.0 0.0 ${(base_height + voxel_width)/2}" rpy="0.0 0.0 0.0"/>
+    </xacro:voxel>
 </robot>

File: src/floatbot_description/urdf/floatbot_base.urdf.xacro (robot description, xacro)
@@ -2,5 +2,5 @@
 <robot xmlns:xacro="http://www.ros.org/wiki/xacro">
     <xacro:property name="base_diameter" value=".3"/>
-    <xacro:property name="base_height" value=".48"/>
+    <xacro:property name="base_height" value=".475"/>
     <xacro:macro name="floatbot_base" params="prefix">
         <link name="${prefix}base_footprint"/>
@@ -13,17 +13,10 @@
                     <color rgba="0.0 0.0 1.0 1.0"/>
                 </material>
-                <origin xyz="0.0 0.0 0.0" rpy="0.0 0.0 0.0"/>
             </visual>
-            <collision>
-                <geometry>
-                    <cylinder radius="${base_diameter/2}" length="${base_height}"/>
-                </geometry>
-                <origin xyz="0.0 0.0 0.0" rpy="0.0 0.0 0.0"/>
-            </collision>
         </link>
         <joint name="${prefix}base_joint" type="fixed">
+            <origin xyz="0.0 0.0 ${(base_height)/2}" rpy="0.0 0.0 0.0"/>
             <parent link="${prefix}base_footprint"/>
             <child link="${prefix}base_link"/>
-            <origin xyz="0.0 0.0 ${base_height/2}" rpy="0.0 0.0 0.0"/>
         </joint>
     </xacro:macro>

Commit message: Implemented apriltag description

File: src/floatbot_description/urdf/floatbot.urdf.xacro (robot description, xacro)
@@ -5,11 +5,11 @@
     <xacro:include filename="$(find floatbot_description)/urdf/floatbot_base.urdf.xacro"/>
     <xacro:include filename="$(find floatbot_description)/urdf/voxel.urdf.xacro"/>
-    <xacro:floatbot_base
-        prefix="$(arg prefix)"
-    />
-    <xacro:voxel
-        prefix="$(arg prefix)"
-        parent="$(arg prefix)base_link">
+    <xacro:include filename="$(find floatbot_description)/urdf/apriltag.urdf.xacro"/>
+    <xacro:floatbot_base prefix="$(arg prefix)"/>
+    <xacro:voxel prefix="$(arg prefix)" parent="$(arg prefix)base_link">
         <origin xyz="0.0 0.0 ${(base_height + voxel_width)/2}" rpy="0.0 0.0 0.0"/>
     </xacro:voxel>
+    <xacro:apriltag prefix="$(arg prefix)" tag_id="0" tag_size=".142" parent="$(arg prefix)voxel_link">
+        <origin xyz="0.0 0.0 ${(voxel_width)/2}" rpy="0.0 0.0 0.0"/>
+    </xacro:apriltag>
 </robot>

File: src/floatbot_description/urdf/floatbot_base.urdf.xacro (robot description, xacro)
@@ -1,4 +1,4 @@
 <?xml version="1.0" encoding="UTF-8"?>
-<robot xmlns:xacro="http://www.ros.org/wiki/xacro">
+<robot xmlns:xacro="http://www.ros.org/wiki/xacro" name="floatbot_base">
     <xacro:property name="base_diameter" value=".3"/>
     <xacro:property name="base_height" value=".475"/>

File: src/floatbot_description/urdf/voxel.urdf.xacro (robot description, xacro)
@@ -1,4 +1,4 @@
 <?xml version="1.0" encoding="UTF-8"?>
-<robot xmlns:xacro="http://www.ros.org/wiki/xacro">
+<robot xmlns:xacro="http://www.ros.org/wiki/xacro" name="voxel">
     <xacro:property name="voxel_width" value=".305"/>
     <xacro:macro name="voxel" params="prefix parent *origin">
