Commit message: Fixed a bug with floatbot description parameters

File: src/floatbot_description/urdf/apriltag.urdf.xacro (robot description, xacro)
@@ -3,5 +3,5 @@
     <xacro:property name="tag_width" value=".003"/>
     <xacro:macro name="apriltag" params="prefix tag_id tag_size parent *origin">
-        <link name="${prefix}tag_{tag_id}_link">
+        <link name="${prefix}tag_${tag_id}_link">
             <visual>
                 <geometry>
@@ -13,8 +13,8 @@
             </visual>
         </link>
-        <joint name="${prefix}tag_{tag_id}_joint" type="fixed">
+        <joint name="${prefix}tag_${tag_id}_joint" type="fixed">
             <xacro:insert_block name="origin"/>
             <parent link="${prefix}${parent}"/>
-            <child link="${prefix}tag_{tag_id}_link"/>
+            <child link="${prefix}tag_${tag_id}_link"/>
         </joint>
     </xacro:macro>

File: src/floatbot_description/urdf/floatbot.urdf.xacro (robot description, xacro)
@@ -3,4 +3,5 @@
     <xacro:arg name="robot_name" default="floatbot"/>
     <xacro:arg name="prefix" default=""/>
+    <xacro:arg name="tag_id" default="1"/>
     <xacro:include filename="$(find floatbot_description)/urdf/floatbot_base.urdf.xacro"/>
     <xacro:include filename="$(find floatbot_description)/urdf/voxel.urdf.xacro"/>
@@ -10,5 +11,5 @@
         <origin xyz="0.0 0.0 ${(base_height + voxel_width)/2}" rpy="0.0 0.0 0.0"/>
     </xacro:voxel>
-    <xacro:apriltag prefix="$(arg prefix)" tag_id="0" tag_size=".142" parent="$(arg prefix)voxel_link">
+    <xacro:apriltag prefix="$(arg prefix)" tag_id="$(arg tag_id)" tag_size=".142" parent="$(arg prefix)voxel_link">
         <origin xyz="0.0 0.0 ${(voxel_width)/2}" rpy="0.0 0.0 0.0"/>
     </xacro:apriltag>
